Commit message: proper namespacing

File: riptide_descriptions/robots/talos.xacro (robot description, xacro)
@@ -1,11 +1,11 @@
 <?xml version="1.0"?>
-<robot name="tempest" xmlns:xacro="http://www.ros.org/wiki/xacro" >
+<robot name="talos" xmlns:xacro="http://www.ros.org/wiki/xacro" >
   <xacro:arg name="debug" default="0"/>
-  <xacro:arg name="namespace" default="tempest"/>
+  <xacro:arg name="namespace" default="talos"/>
   <xacro:arg name="inertial_reference_frame" default="world"/>
   <!-- Include the Robot macro file -->
   <xacro:include filename="$(find riptide_descriptions2)/urdf/robot_base.xacro"/>
   <!-- Read the config -->
-  <xacro:property name="yaml_file" value="$(find riptide_descriptions2)/config/tempest.yaml" />
+  <xacro:property name="yaml_file" value="$(find riptide_descriptions2)/config/talos.yaml" />
   <xacro:property name="config" value="${load_yaml(yaml_file)}"/>
   <xacro:property name="body_file" value="package://riptide_descriptions2/meshes/Tempest.dae"/>

Commit message: confirm sensor and thruster positions on talos

File: riptide_descriptions/robots/talos.xacro (robot description, xacro)
@@ -9,5 +9,5 @@
   <xacro:property name="yaml_file" value="$(find riptide_descriptions2)/config/talos.yaml" />
   <xacro:property name="config" value="${load_yaml(yaml_file)}"/>
-  <xacro:property name="body_file" value="package://riptide_descriptions2/meshes/Tempest.dae"/>
+  <xacro:property name="body_file" value="package://riptide_descriptions2/meshes/Talos.dae"/>
   <xacro:property name="prop_file" value="package://riptide_descriptions2/meshes/Propeller.dae"/>
   <!-- Create robot -->

File: riptide_descriptions/urdf/robot_actuators.xacro (robot description, xacro)
@@ -42,9 +42,4 @@
       <xacro:dummy_inertia />
       <xacro:no_collision />
-      <visual>
-        <geometry>
-          <box size="0.2 0.05 0.05"/>
-        </geometry>
-      </visual>
     </link>
   </xacro:macro>
@@ -60,9 +55,4 @@
       <xacro:dummy_inertia />
       <xacro:no_collision />
-      <visual>
-        <geometry>
-          <box size="0.25 0.05 0.05"/>
-        </geometry>
-      </visual>
     </link>
   </xacro:macro>
@@ -78,9 +68,4 @@
       <xacro:dummy_inertia />
       <xacro:no_collision />
-      <visual>
-        <geometry>
-          <box size="0.025 0.025 0.1"/>
-        </geometry>
-      </visual>
     </link>
   </xacro:macro>
