Commit message: scoped namespacing, update puddles information

File: riptide_descriptions/robots/puddles.xacro (robot description, xacro)
@@ -9,6 +9,6 @@
   <xacro:property name="yaml_file" value="$(find riptide_descriptions2)/config/puddles.yaml" />
   <xacro:property name="config" value="${load_yaml(yaml_file)}"/>
-  <xacro:property name="body_file" value="$(find riptide_descriptions2)/meshes/Puddles.dae"/>
-  <xacro:property name="prop_file" value="$(find riptide_descriptions2)/meshes/Propeller.dae"/>
+  <xacro:property name="body_file" value="package://riptide_descriptions2/meshes/Puddles.dae"/>
+  <xacro:property name="prop_file" value="package://riptide_descriptions2/meshes/Propeller.dae"/>
   <!-- Create robot -->
   <xacro:robot_base
