Commit message: puddles post pool test

File: riptide_descriptions/urdf/robot_sensors.xacro (robot description, xacro)
@@ -49,13 +49,22 @@
     <xacro:if value="${cameras != []}">
       <xacro:property name="camera" value="${cameras[0]}"/>
+      <link name="${namespace}/${camera['name']}_base_link">
+        <xacro:dummy_inertia/>
+        <xacro:no_collision/>
+      </link>
+      <joint name="${namespace}/${camera['name']}_joint" type="fixed">
+        <parent link="${namespace}/origin"/>
+        <child link="${namespace}/${camera['name']}_base_link"/>
+        <origin xyz="${camera['pose'][0]} ${camera['pose'][1]} ${camera['pose'][2]}"
+                rpy="${camera['pose'][3]} ${camera['pose'][4]} ${camera['pose'][5]}"/>
+      </joint>
       <!-- Stereo Camera(s) -->
       <xacro:if value="${camera['type'] == 'stereo'}">
         <xacro:stereo_macro
           namespace="${namespace}"
-          parent_link="${namespace}/origin"
+          parent_link="${namespace}/${camera['name']}_base_link"
           name="${camera['name']}"
           baseline="${camera['baseline']}">
-          <origin xyz="${camera['pose'][0]} ${camera['pose'][1]} ${camera['pose'][2]}"
-                  rpy="${camera['pose'][3]} ${camera['pose'][4]} ${camera['pose'][5]}"/>
+          <origin xyz="0 ${camera['baseline'] / 2} 0" />
         </xacro:stereo_macro>
       </xacro:if>

File: riptide_descriptions/urdf/snippets.xacro (robot description, xacro)
@@ -47,5 +47,5 @@
     </xacro:macro>
     <xacro:macro name="stereo_macro" params="namespace parent_link name baseline *origin">
-        <xacro:camera_macro namespace="${namespace}/${name}" name="left" parent_link="${namespace}/origin">
+        <xacro:camera_macro namespace="${namespace}/${name}" name="left" parent_link="${parent_link}">
             <xacro:insert_block name="origin" />
         </xacro:camera_macro>

Commit message: make zed play in tf

File: riptide_descriptions/urdf/robot_sensors.xacro (robot description, xacro)
@@ -83,4 +83,14 @@
         <!-- Suffix isn't set here because right now we just have one, but you should just need to change the suffix for each and it'll work. -->
         <xacro:unless value="${camera['type'] == 'mono'}">
+          <xacro:if value="${camera['type'] == 'zed'}">
+          <!-- TODO: zed macro is not needed when we figure out how to change the name of hte zed base link-->
+            <xacro:zed_macro
+             namespace="${namespace}"
+             name="${camera['name']}"
+             parent_link="${namespace}/origin">
+             <origin xyz="${camera['pose'][0]} ${camera['pose'][1]} ${camera['pose'][2]}"
+                    rpy="${camera['pose'][3]} ${camera['pose'][4]} ${camera['pose'][5]}"/>
+            </xacro:zed_macro>
+          </xacro:if>
         </xacro:unless>
       </xacro:unless>

File: riptide_descriptions/urdf/snippets.xacro (robot description, xacro)
@@ -53,4 +53,12 @@
             <origin xyz="0 ${-baseline} 0" />
         </xacro:camera_macro>
+    </xacro:macro>
+    <xacro:macro name="zed_macro" params="namespace parent_link name *origin">
+        <link name="${name}" />
+        <joint name="${namespace}/${name}_origin_joint" type="fixed">
+            <parent link="${parent_link}" />
+            <child link="${name}" />
+            <xacro:insert_block name="origin" />
+        </joint>
     </xacro:macro>
     <xacro:macro name="dvl_plugin_macro" params="namespace suffix parent_link *origin">

Commit message: added dfc to urdf and made zed better

File: riptide_descriptions/urdf/robot_sensors.xacro (robot description, xacro)
@@ -49,11 +49,12 @@
     <xacro:if value="${cameras != []}">
       <xacro:property name="camera" value="${cameras[0]}"/>
-      <link name="${namespace}/${camera['name']}_base_link">
+      <xacro:property name="camera_base_link" value="${namespace}/${camera['name']}_base_link"/>
+      <link name="${camera_base_link}">
         <xacro:dummy_inertia/>
         <xacro:no_collision/>
       </link>
-      <joint name="${namespace}/${camera['name']}_joint" type="fixed">
+      <joint name="${camera_base_link}_joint" type="fixed">
         <parent link="${namespace}/origin"/>
-        <child link="${namespace}/${camera['name']}_base_link"/>
+        <child link="${camera_base_link}"/>
         <origin xyz="${camera['pose'][0]} ${camera['pose'][1]} ${camera['pose'][2]}"
                 rpy="${camera['pose'][3]} ${camera['pose'][4]} ${camera['pose'][5]}"/>
@@ -84,12 +85,8 @@
         <xacro:unless value="${camera['type'] == 'mono'}">
           <xacro:if value="${camera['type'] == 'zed'}">
-          <!-- TODO: zed macro is not needed when we figure out how to change the name of hte zed base link-->
+          <!-- TODO: zed macro is not needed when we figure out how to change the name of the zed base link-->
             <xacro:zed_macro
              namespace="${namespace}"
-             name="${camera['name']}"
-             parent_link="${namespace}/origin">
-             <origin xyz="${camera['pose'][0]} ${camera['pose'][1]} ${camera['pose'][2]}"
-                    rpy="${camera['pose'][3]} ${camera['pose'][4]} ${camera['pose'][5]}"/>
-            </xacro:zed_macro>
+             parent_link="${camera_base_link}" />
           </xacro:if>
         </xacro:unless>

File: riptide_descriptions/urdf/snippets.xacro (robot description, xacro)
@@ -54,10 +54,14 @@
         </xacro:camera_macro>
     </xacro:macro>
-    <xacro:macro name="zed_macro" params="namespace parent_link name *origin">
-        <link name="${name}" />
-        <joint name="${namespace}/${name}_origin_joint" type="fixed">
+    <xacro:macro name="zed_macro" params="namespace parent_link">
+        <!-- this link must be called "zed_camera_link" because thats what the zed launch attaches its tree to -->
+        <link name="zed_camera_link">
+            <xacro:dummy_inertia/>
+            <xacro:no_collision/>
+        </link>
+        <joint name="${namespace}/zed_camera_link_origin_joint" type="fixed">
             <parent link="${parent_link}" />
-            <child link="${name}" />
-            <xacro:insert_block name="origin" />
+            <child link="zed_camera_link" />
+            <origin xyz="0 0 0" rpy="0 0 0"/>
         </joint>
     </xacro:macro>

Commit message: integrate zed into navigation launch

File: riptide_descriptions/urdf/robot_sensors.xacro (robot description, xacro)
@@ -85,7 +85,7 @@
         <xacro:unless value="${camera['type'] == 'mono'}">
           <xacro:if value="${camera['type'] == 'zed'}">
-          <!-- TODO: zed macro is not needed when we figure out how to change the name of the zed base link-->
             <xacro:zed_macro
              namespace="${namespace}"
+             name="talos/${camera['name']}_link"
              parent_link="${camera_base_link}" />
           </xacro:if>

File: riptide_descriptions/urdf/snippets.xacro (robot description, xacro)
@@ -54,7 +54,6 @@
         </xacro:camera_macro>
     </xacro:macro>
-    <xacro:macro name="zed_macro" params="namespace parent_link">
-        <!-- this link must be called "zed_camera_link" because thats what the zed launch attaches its tree to -->
-        <link name="zed_camera_link">
+    <xacro:macro name="zed_macro" params="namespace name parent_link">
+        <link name="${name}">
             <xacro:dummy_inertia/>
             <xacro:no_collision/>
@@ -62,5 +61,5 @@
         <joint name="${namespace}/zed_camera_link_origin_joint" type="fixed">
             <parent link="${parent_link}" />
-            <child link="zed_camera_link" />
+            <child link="${name}" />
             <origin xyz="0 0 0" rpy="0 0 0"/>
         </joint>

Commit message: Acoustics Measurement

File: riptide_descriptions/urdf/robot_sensors.xacro (robot description, xacro)
@@ -27,4 +27,22 @@
     </xacro:pressure_plugin_macro>
   <!-- </xacro:if> -->
+  <!-- port acoustic pod -->
+  <xacro:property name="acoustics_port" value="${config['acoustics']['port']}"/>
+    <xacro:pressure_plugin_macro
+      namespace="${namespace}"
+      suffix=""
+      parent_link="${namespace}/origin">
+      <origin xyz="${acoustics_port['pose'][0]} ${acoustics_port['pose'][1]} ${acoustics_port['pose'][2]}"
+              rpy="${acoustics_port['pose'][3]} ${acoustics_port['pose'][4]} ${acoustics_port['pose'][5]}"/>
+    </xacro:pressure_plugin_macro>
+  <!--starboard acoustic pod-->
+  <xacro:property name="acoustics_starboard" value="${config['acoustics']['starboard']}"/>
+  <xacro:pressure_plugin_macro
+    namespace="${namespace}"
+    suffix=""
+    parent_link="${namespace}/origin">
+    <origin xyz="${acoustics_starboard['pose'][0]} ${acoustics_starboard['pose'][1]} ${acoustics_starboard['pose'][2]}"
+            rpy="${acoustics_starboard['pose'][3]} ${acoustics_starboard['pose'][4]} ${acoustics_starboard['pose'][5]}"/>
+  </xacro:pressure_plugin_macro>
   <!-- IMU  -->
   <!-- TODO: Get imu model from config -->

Commit message: Added changes

File: riptide_descriptions/urdf/robot_sensors.xacro (robot description, xacro)
@@ -29,20 +29,20 @@
   <!-- port acoustic pod -->
   <xacro:property name="acoustics_port" value="${config['acoustics']['port']}"/>
-    <xacro:pressure_plugin_macro
+    <xacro:acoustics_plugin_macro
       namespace="${namespace}"
-      suffix=""
+      suffix="_port"
       parent_link="${namespace}/origin">
       <origin xyz="${acoustics_port['pose'][0]} ${acoustics_port['pose'][1]} ${acoustics_port['pose'][2]}"
               rpy="${acoustics_port['pose'][3]} ${acoustics_port['pose'][4]} ${acoustics_port['pose'][5]}"/>
-    </xacro:pressure_plugin_macro>
+    </xacro:acoustics_plugin_macro>
   <!--starboard acoustic pod-->
   <xacro:property name="acoustics_starboard" value="${config['acoustics']['starboard']}"/>
-  <xacro:pressure_plugin_macro
+  <xacro:acoustics_plugin_macro
     namespace="${namespace}"
-    suffix=""
+    suffix="_starboard"
     parent_link="${namespace}/origin">
     <origin xyz="${acoustics_starboard['pose'][0]} ${acoustics_starboard['pose'][1]} ${acoustics_starboard['pose'][2]}"
             rpy="${acoustics_starboard['pose'][3]} ${acoustics_starboard['pose'][4]} ${acoustics_starboard['pose'][5]}"/>
-  </xacro:pressure_plugin_macro>
+    </xacro:acoustics_plugin_macro>
   <!-- IMU  -->
   <!-- TODO: Get imu model from config -->

File: riptide_descriptions/urdf/snippets.xacro (robot description, xacro)
@@ -91,4 +91,17 @@
         </joint>
     </xacro:macro>
+    <xacro:macro name="acoustics_plugin_macro" params="namespace suffix parent_link *origin">
+        <link name="${namespace}/acoustics${suffix}_link">
+            <xacro:dummy_inertia />
+            <xacro:no_collision />
+        </link>
+        <joint name="${namespace}/acoustics${suffix}_joint" type="revolute">
+            <xacro:insert_block name="origin" />
+            <parent link="${parent_link}" />
+            <child link="${namespace}/acoustics${suffix}_link" />
+            <limit upper="0" lower="0" effort="0" velocity="0" />
+            <axis xyz="1 0 0" />
+        </joint>
+    </xacro:macro>
     <xacro:macro name="imu_plugin_macro" params="namespace imu_suffix parent_link *origin">
         <!-- IMU link -->

Commit message: Fixed Config to For Acoustics & Tf in Matlab

File: riptide_descriptions/urdf/robot_sensors.xacro (robot description, xacro)
@@ -27,4 +27,22 @@
     </xacro:pressure_plugin_macro>
   <!-- </xacro:if> -->
+  <!-- port acoustic pod -->
+  <xacro:property name="acoustics_port" value="${config['acoustics']['port']}"/>
+  <xacro:acoustics_plugin_macro
+    namespace="${namespace}"
+    suffix="_port"
+    parent_link="${namespace}/origin">
+    <origin xyz="${acoustics_port['pose'][0]} ${acoustics_port['pose'][1]} ${acoustics_port['pose'][2]}"
+            rpy="${acoustics_port['pose'][3]} ${acoustics_port['pose'][4]} ${acoustics_port['pose'][5]}"/>
+  </xacro:acoustics_plugin_macro>
+  <!--starboard acoustic pod-->
+  <xacro:property name="acoustics_starboard" value="${config['acoustics']['starboard']}"/>
+  <xacro:acoustics_plugin_macro
+  namespace="${namespace}"
+  suffix="_starboard"
+  parent_link="${namespace}/origin">
+  <origin xyz="${acoustics_starboard['pose'][0]} ${acoustics_starboard['pose'][1]} ${acoustics_starboard['pose'][2]}"
+          rpy="${acoustics_starboard['pose'][3]} ${acoustics_starboard['pose'][4]} ${acoustics_starboard['pose'][5]}"/>
+  </xacro:acoustics_plugin_macro>
   <!-- IMU  -->
   <!-- TODO: Get imu model from config -->

File: riptide_descriptions/urdf/snippets.xacro (robot description, xacro)
@@ -91,4 +91,17 @@
         </joint>
     </xacro:macro>
+    <xacro:macro name="acoustics_plugin_macro" params="namespace suffix parent_link *origin">
+    <link name="${namespace}/acoustics${suffix}_link">
+        <xacro:dummy_inertia />
+        <xacro:no_collision />
+    </link>
+    <joint name="${namespace}/acoustics${suffix}_joint" type="revolute">
+        <xacro:insert_block name="origin" />
+        <parent link="${parent_link}" />
+        <child link="${namespace}/acoustics${suffix}_link" />
+        <limit upper="0" lower="0" effort="0" velocity="0" />
+        <axis xyz="1 0 0" />
+    </joint>
+    </xacro:macro>
     <xacro:macro name="imu_plugin_macro" params="namespace imu_suffix parent_link *origin">
         <!-- IMU link -->

Commit message: both cameras working now. still need to double check poses

File: riptide_descriptions/urdf/robot_sensors.xacro (robot description, xacro)
@@ -105,5 +105,5 @@
             <xacro:zed_macro
              namespace="${namespace}"
-             name="talos/${camera['name']}_link"
+             name="talos/${camera['name']}"
              parent_link="${camera_base_link}" />
           </xacro:if>

File: riptide_descriptions/urdf/snippets.xacro (robot description, xacro)
@@ -55,11 +55,11 @@
     </xacro:macro>
     <xacro:macro name="zed_macro" params="namespace name parent_link">
-        <link name="${name}">
-            <xacro:dummy_inertia/>
-            <xacro:no_collision/>
+        <link name="${name}_camera_link">
+            <xacro:dummy_inertia />
+            <xacro:no_collision />
         </link>
-        <joint name="${namespace}/zed_camera_link_origin_joint" type="fixed">
+        <joint name="${namespace}/${name}_origin_joint" type="fixed">
             <parent link="${parent_link}" />
-            <child link="${name}" />
+            <child link="${name}_camera_link" />
             <origin xyz="0 0 0" rpy="0 0 0"/>
         </joint>

Commit message: Fog No Upside Down

File: riptide_descriptions/urdf/robot_sensors.xacro (robot description, xacro)
@@ -45,4 +45,11 @@
           rpy="${acoustics_starboard['pose'][3]} ${acoustics_starboard['pose'][4]} ${acoustics_starboard['pose'][5]}"/>
   </xacro:acoustics_plugin_macro>
+  <xacro:property name="fog" value="${config['fog']}"/>
+  <xacro:fog_plugin_macro
+  namespace="${namespace}"
+  parent_link="${namespace}/origin">
+  <origin xyz="${fog['pose'][0]} ${fog['pose'][1]} ${fog['pose'][2]}"
+          rpy="${fog['pose'][3]} ${fog['pose'][4]} ${fog['pose'][5]}"/>
+  </xacro:fog_plugin_macro>
   <!-- IMU  -->
   <!-- TODO: Get imu model from config -->

File: riptide_descriptions/urdf/snippets.xacro (robot description, xacro)
@@ -104,4 +104,17 @@
     </joint>
     </xacro:macro>
+    <xacro:macro name="fog_plugin_macro" params="namespace parent_link *origin">
+    <link name="${namespace}/fog_link">
+        <xacro:dummy_inertia />
+        <xacro:no_collision />
+    </link>
+    <joint name="${namespace}/fog_joint" type="revolute">
+        <xacro:insert_block name="origin" />
+        <parent link="${parent_link}" />
+        <child link="${namespace}/fog_link" />
+        <limit upper="0" lower="0" effort="0" velocity="0" />
+        <axis xyz="1 0 0" />
+    </joint>
+    </xacro:macro>
     <xacro:macro name="imu_plugin_macro" params="namespace imu_suffix parent_link *origin">
         <!-- IMU link -->
