Commit message: maybe made xacro more modular but need to test on bot

File: riptide_descriptions/urdf/robot_sensors.xacro (robot description, xacro)
@@ -2,29 +2,31 @@
 <robot xmlns:xacro="http://www.ros.org/wiki/xacro" >
   <!-- Everything here is ENU frame -->
+  <!-- DVL  -->
   <xacro:property name="dvl" value="${config['dvl']}"/>
-  <!-- DVL  -->
-  <!-- TODO: restore below if when xacro releases 1.14.4 -->
-  <!-- <xacro:if value="${'dvl' in config}"> -->
-    <xacro:property name="dvl" value="${config['dvl']}"/>
-    <xacro:dvl_plugin_macro
-      namespace="${namespace}"
-      suffix=""
-      parent_link="${namespace}/origin">
-      <origin xyz="${dvl['pose'][0]} ${dvl['pose'][1]} ${dvl['pose'][2]}"
-              rpy="${dvl['pose'][3]} ${dvl['pose'][4]} ${dvl['pose'][5]}"/>
-    </xacro:dvl_plugin_macro>
-  <!-- </xacro:if> -->
+  <xacro:dvl_plugin_macro
+    namespace="${namespace}"
+    suffix=""
+    parent_link="${namespace}/origin">
+    <origin xyz="${dvl['pose'][0]} ${dvl['pose'][1]} ${dvl['pose'][2]}"
+            rpy="${dvl['pose'][3]} ${dvl['pose'][4]} ${dvl['pose'][5]}"/>
+  </xacro:dvl_plugin_macro>
   <!-- Pressure  -->
-  <!-- TODO: restore below if when xacro releases 1.14.4 -->
-  <!-- <xacro:if value="${'depth' in config}"> -->
-    <xacro:property name="depth" value="${config['depth']}"/>
-    <xacro:pressure_plugin_macro
-      namespace="${namespace}"
-      suffix=""
-      parent_link="${namespace}/origin">
-      <origin xyz="${depth['pose'][0]} ${depth['pose'][1]} ${depth['pose'][2]}"
-              rpy="${depth['pose'][3]} ${depth['pose'][4]} ${depth['pose'][5]}"/>
-    </xacro:pressure_plugin_macro>
-  <!-- </xacro:if> -->
+  <xacro:property name="depth" value="${config['depth']}"/>
+  <xacro:pressure_plugin_macro
+    namespace="${namespace}"
+    suffix=""
+    parent_link="${namespace}/origin">
+    <origin xyz="${depth['pose'][0]} ${depth['pose'][1]} ${depth['pose'][2]}"
+            rpy="${depth['pose'][3]} ${depth['pose'][4]} ${depth['pose'][5]}"/>
+  </xacro:pressure_plugin_macro>
+  <!-- Fog -->
+  <xacro:property name="fog" value="${config['fog']}" />
+  <xacro:fog_macro
+    namespace="${namespace}"
+    suffix=""
+    parent_link="${namespace}/origin">
+    <origin xyz="${fog['pose'][0]} ${fog['pose'][1]} ${fog['pose'][2]}"
+            rpy="${fog['pose'][3]} ${fog['pose'][4]} ${fog['pose'][5]}"/>
+  </xacro:fog_macro>
   <!-- port acoustic pod -->
   <xacro:property name="acoustics_port" value="${config['acoustics']['port']}"/>
@@ -39,9 +41,9 @@
   <xacro:property name="acoustics_starboard" value="${config['acoustics']['starboard']}"/>
   <xacro:acoustics_plugin_macro
-  namespace="${namespace}"
-  suffix="_starboard"
-  parent_link="${namespace}/origin">
-  <origin xyz="${acoustics_starboard['pose'][0]} ${acoustics_starboard['pose'][1]} ${acoustics_starboard['pose'][2]}"
-          rpy="${acoustics_starboard['pose'][3]} ${acoustics_starboard['pose'][4]} ${acoustics_starboard['pose'][5]}"/>
+    namespace="${namespace}"
+    suffix="_starboard"
+    parent_link="${namespace}/origin">
+    <origin xyz="${acoustics_starboard['pose'][0]} ${acoustics_starboard['pose'][1]} ${acoustics_starboard['pose'][2]}"
+            rpy="${acoustics_starboard['pose'][3]} ${acoustics_starboard['pose'][4]} ${acoustics_starboard['pose'][5]}"/>
   </xacro:acoustics_plugin_macro>
   <!-- IMU  -->
@@ -61,6 +63,5 @@
   <xacro:default_pose_3d_macro
     namespace="${namespace}"
-    parent_link="${namespace}/base_link"
-    inertial_reference_frame="${inertial_reference_frame}" />
+    parent_link="${namespace}/base_link" />
   <!-- Builds any number of cameras from yaml -->
   <xacro:macro name="cameras_macro" params="namespace cameras">
@@ -101,9 +102,10 @@
         <!-- MYNT/ZED Camera -->
         <!-- Suffix isn't set here because right now we just have one, but you should just need to change the suffix for each and it'll work. -->
+        <!-- name="talos/${camera['name']}_link" -->
         <xacro:unless value="${camera['type'] == 'mono'}">
           <xacro:if value="${camera['type'] == 'zed'}">
             <xacro:zed_macro
              namespace="${namespace}"
-             name="talos/${camera['name']}_link"
+             name="${camera['name']}"
              parent_link="${camera_base_link}" />
           </xacro:if>

File: riptide_descriptions/urdf/snippets.xacro (robot description, xacro)
@@ -16,19 +16,30 @@
         </collision>
     </xacro:macro>
+    <xacro:macro name="generic_frame_macro" params="namespace name suffix parent_link *origin">
+        <link name="${namespace}/${name}${suffix}_link">
+            <xacro:dummy_inertia />
+            <xacro:no_collision />
+        </link>
+        <joint name="${namespace}/${name}${suffix}_joint" type="fixed">
+            <xacro:insert_block name="origin" />
+            <parent link="${parent_link}" />
+            <child link="${namespace}/${name}${suffix}_link" />
+            <limit upper="0" lower="0" effort="0" velocity="0" />
+            <axis xyz="1 0 0" />
+        </joint>
+    </xacro:macro>
     <!-- Ground truth position -->
-    <xacro:macro name="default_pose_3d_macro" params="namespace parent_link inertial_reference_frame">
+    <xacro:macro name="default_pose_3d_macro" params="namespace parent_link">
         <!-- Mount a 3D pose sensor -->
-        <link name="${namespace}/pose_sensor_link">
-            <xacro:dummy_inertia />
-        </link>
-        <joint name="${namespace}/pose_sensor_joint" type="revolute">
-            <axis xyz="0 0 1" />
-            <parent link="${parent_link}" />
-            <child link="${namespace}/pose_sensor_link" />
-            <limit effort="0" lower="0" upper="0" velocity="0" />
-        </joint>
+        <xacro:generic_frame_macro
+            namespace="${namespace}"
+            name="pose_sensor"
+            suffix=""
+            parent_link="${parent_link}">
+            <origin xyz="0 0 0" rpy="0 0 0" />
+        </xacro:generic_frame_macro>
     </xacro:macro>
     <xacro:macro name="camera_macro" params="namespace name parent_link *origin">
-        <link name="${namespace}/${name}_link">
+        <!-- <link name="${namespace}/${name}_link">
             <xacro:dummy_inertia />
             <xacro:no_collision />
@@ -38,5 +49,13 @@
             <parent link="${parent_link}" />
             <child link="${namespace}/${name}_link" />
-        </joint>
+        </joint> -->
+        <xacro:generic_frame_macro
+            namespace="${namespace}"
+            name="${name}"
+            suffix=""
+            parent_link="${parent_link}">
+            <xacro:insert_block name="origin" />
+        </xacro:generic_frame_macro>
+<!--
         <link name="${namespace}/${name}_optical" />
         <joint name="${namespace}/${name}_optical_joint" type="fixed">
@@ -44,5 +63,12 @@
             <child link="${namespace}/${name}_optical" />
             <origin rpy="${-pi/2} 0 ${-pi/2}"></origin>
-        </joint>
+        </joint> -->
+        <xacro:generic_frame_macro
+            namespace="${namespace}"
+            name="${name}_optical"
+            suffix=""
+            parent_link="${namespace}/${name}_link">
+            <origin rpy="${-pi/2} 0 ${-pi/2}"></origin>
+        </xacro:generic_frame_macro>
     </xacro:macro>
     <xacro:macro name="stereo_macro" params="namespace parent_link name baseline *origin">
@@ -55,5 +81,5 @@
     </xacro:macro>
     <xacro:macro name="zed_macro" params="namespace name parent_link">
-        <link name="${name}">
+        <!-- <link name="${name}">
             <xacro:dummy_inertia/>
             <xacro:no_collision/>
@@ -63,8 +89,15 @@
             <child link="${name}" />
             <origin xyz="0 0 0" rpy="0 0 0"/>
-        </joint>
+        </joint> -->
+        <xacro:generic_frame_macro
+            namespace="${namespace}"
+            name="${name}"
+            suffix=""
+            parent_link="${parent_link}">
+            <origin xyz="0 0 0" rpy="0 0 0"/>
+        </xacro:generic_frame_macro>
     </xacro:macro>
     <xacro:macro name="dvl_plugin_macro" params="namespace suffix parent_link *origin">
-        <link name="${namespace}/dvl${suffix}_link">
+        <!-- <link name="${namespace}/dvl${suffix}_link">
             <xacro:dummy_inertia />
             <xacro:no_collision />
@@ -76,8 +109,15 @@
             <limit upper="0" lower="0" effort="0" velocity="0" />
             <axis xyz="1 0 0" />
-        </joint>
+        </joint> -->
+        <xacro:generic_frame_macro
+            namespace="${namespace}"
+            name="dvl"
+            suffix="${suffix}"
+            parent_link="${parent_link}">
+            <xacro:insert_block name="origin" />
+        </xacro:generic_frame_macro>
     </xacro:macro>
     <xacro:macro name="pressure_plugin_macro" params="namespace suffix parent_link *origin">
-        <link name="${namespace}/pressure${suffix}_link">
+        <!-- <link name="${namespace}/pressure${suffix}_link">
             <xacro:dummy_inertia />
             <xacro:no_collision />
@@ -89,33 +129,63 @@
             <limit upper="0" lower="0" effort="0" velocity="0" />
             <axis xyz="1 0 0" />
-        </joint>
+        </joint> -->
+        <xacro:generic_frame_macro
+            namespace="${namespace}"
+            name="pressure"
+            suffix="${suffix}"
+            parent_link="${parent_link}">
+            <xacro:insert_block name="origin" />
+        </xacro:generic_frame_macro>
+    </xacro:macro>
+    <xacro:macro name="fog_macro" params="namespace suffix parent_link *origin">
+        <xacro:insert_block name="origin" />
+        <xacro:generic_frame_macro
+            namespace="${namespace}"
+            name="fog"
+            suffix="${suffix}"
+            parent_link="${parent_link}">
+            <xacro:insert_block name="origin" />
+        </xacro:generic_frame_macro>
     </xacro:macro>
     <xacro:macro name="acoustics_plugin_macro" params="namespace suffix parent_link *origin">
-    <link name="${namespace}/acoustics${suffix}_link">
-        <xacro:dummy_inertia />
-        <xacro:no_collision />
-    </link>
-    <joint name="${namespace}/acoustics${suffix}_joint" type="revolute">
-        <xacro:insert_block name="origin" />
-        <parent link="${parent_link}" />
-        <child link="${namespace}/acoustics${suffix}_link" />
-        <limit upper="0" lower="0" effort="0" velocity="0" />
-        <axis xyz="1 0 0" />
-    </joint>
+        <!-- <link name="${namespace}/acoustics${suffix}_link">
+            <xacro:dummy_inertia />
+            <xacro:no_collision />
+        </link>
+        <joint name="${namespace}/acoustics${suffix}_joint" type="revolute">
+            <xacro:insert_block name="origin" />
+            <parent link="${parent_link}" />
+            <child link="${namespace}/acoustics${suffix}_link" />
+            <limit upper="0" lower="0" effort="0" velocity="0" />
+            <axis xyz="1 0 0" />
+        </joint> -->
+        <xacro:generic_frame_macro
+            namespace="${namespace}"
+            name="acoustics"
+            suffix="${suffix}"
+            parent_link="${parent_link}">
+            <xacro:insert_block name="origin" />
+        </xacro:generic_frame_macro>
     </xacro:macro>
     <xacro:macro name="imu_plugin_macro" params="namespace imu_suffix parent_link *origin">
-        <!-- IMU link -->
+        <!-- IMU link
         <link name="${namespace}/imu${imu_suffix}_link">
             <xacro:dummy_inertia />
         </link>
-        <link name="${namespace}/imu${imu_suffix}_revolute_link">
-            <xacro:dummy_inertia />
-        </link>
-        <!-- IMU joint -->
         <joint name="${namespace}/imu${imu_suffix}_joint" type="fixed">
             <xacro:insert_block name="origin" />
             <parent link="${parent_link}" />
             <child link="${namespace}/imu${imu_suffix}_link" />
-        </joint>
+        </joint> -->
+        <xacro:generic_frame_macro
+            namespace="${namespace}"
+            name="imu"
+            suffix="${imu_suffix}"
+            parent_link="${parent_link}">
+            <xacro:insert_block name="origin" />
+        </xacro:generic_frame_macro>
+        <!-- <link name="${namespace}/imu${imu_suffix}_revolute_link">
+            <xacro:dummy_inertia />
+        </link>
         <joint name="${namespace}/imu${imu_suffix}_revolute_joint" type="revolute">
             <xacro:insert_block name="origin" />
@@ -124,5 +194,12 @@
             <limit upper="0" lower="0" effort="0" velocity="0" />
             <axis xyz="1 0 0" />
-        </joint>
+        </joint> -->
+        <xacro:generic_frame_macro
+            namespace="${namespace}"
+            name="imu${imu_suffix}_revolute"
+            suffix=""
+            parent_link="${parent_link}">
+            <xacro:insert_block name="origin" />
+        </xacro:generic_frame_macro>
     </xacro:macro>
     <xacro:macro name="thruster_macro" params="namespace
