Commit message: add actuators

File: riptide_descriptions/urdf/robot_actuators.xacro (robot description, xacro)
@@ -31,13 +31,13 @@
     </xacro:if>
   </xacro:macro>
-  <xacro:macro name="claw_macro" params="namespace config">
-    <xacro:property name="claw" value="${config['claw']}"/>
-    <joint name="${namespace}/claw_joint" type="fixed">
-      <origin xyz="${claw['pose'][0]} ${claw['pose'][1]} ${claw['pose'][2]}"
-              rpy="${claw['pose'][3]} ${claw['pose'][4]} ${claw['pose'][5]}"/>
+  <xacro:macro name="poker_macro" params="namespace config">
+    <xacro:property name="poker" value="${config['poker']}"/>
+    <joint name="${namespace}/poker_joint" type="fixed">
+      <origin xyz="${poker['pose'][0]} ${poker['pose'][1]} ${poker['pose'][2]}"
+              rpy="${poker['pose'][3]} ${poker['pose'][4]} ${poker['pose'][5]}"/>
       <parent link="${namespace}/origin"/>
-      <child link="${namespace}/claw_link"/>
+      <child link="${namespace}/poker_link"/>
     </joint>
-    <link name="${namespace}/claw_link">
+    <link name="${namespace}/poker_link">
       <xacro:dummy_inertia />
       <xacro:no_collision />
@@ -75,5 +75,5 @@
         thrusters="${config['thrusters']}"
         index="0"/>
-  <xacro:claw_macro
+  <xacro:poker_macro
         namespace="${namespace}"
         config="${config}"/>

Commit message: fix integer overflow issue, remove unneeded xacro things

File: riptide_descriptions/urdf/robot_actuators.xacro (robot description, xacro)
@@ -14,5 +14,5 @@
 <robot xmlns:xacro="http://www.ros.org/wiki/xacro" >
   <!-- Macro makes any number of thrusters from config -->
-  <xacro:macro name="thrusters_macro" params="namespace config thrusters index">
+  <xacro:macro name="thrusters_macro" params="namespace thrusters index">
     <xacro:if value="${thrusters != []}">
       <xacro:property name="thruster" value="${thrusters[0]}"/>
@@ -26,5 +26,4 @@
       <xacro:thrusters_macro
         namespace="${namespace}"
-        config="${config}"
         thrusters="${thrusters[1:]}"
         index="${index+1}"/>
@@ -72,5 +71,4 @@
   <xacro:thrusters_macro
         namespace="${namespace}"
-        config="${config['thruster']}"
         thrusters="${config['thrusters']}"
         index="0"/>

Commit message: add separate torpedo launcher frames

File: riptide_descriptions/urdf/robot_actuators.xacro (robot description, xacro)
@@ -43,4 +43,15 @@
     </link>
   </xacro:macro>
+  <xacro:macro name="launcher_macro" params="namespace name parent *origin">
+    <link name="${namespace}/${name}_link">
+      <xacro:dummy_inertia/>
+      <xacro:no_collision/>
+    </link>
+    <joint name="${namespace}/${name}_joint" type="fixed">
+      <xacro:insert_block name="origin"/>
+      <parent link="${parent}"/>
+      <child link="${namespace}/${name}_link"/>
+    </joint>
+  </xacro:macro>
   <xacro:macro name="torpedo_macro" params="namespace config">
     <xacro:property name="torpedo" value="${config['torpedos']}"/>
@@ -55,4 +66,12 @@
       <xacro:no_collision />
     </link>
+    <xacro:launcher_macro namespace="${namespace}" name="torpedo_0" parent="${namespace}/torpedo_link">
+      <origin xyz="0 ${-torpedo['baseline'] / 2} 0"
+              rpy="0 0 0"/>
+    </xacro:launcher_macro>
+    <xacro:launcher_macro namespace="${namespace}" name="torpedo_1" parent="${namespace}/torpedo_link">
+      <origin xyz="0 ${torpedo['baseline'] / 2} 0"
+              rpy="0 0 0"/>
+    </xacro:launcher_macro>
   </xacro:macro>
   <xacro:macro name="dropper_macro" params="namespace config">

Commit message: Add liltank ekf, and descriptions

File: riptide_descriptions/urdf/robot_actuators.xacro (robot description, xacro)
@@ -55,5 +55,5 @@
   </xacro:macro>
   <xacro:macro name="torpedo_macro" params="namespace config">
-    <xacro:property name="torpedo" value="${config['torpedos']}"/>
+    <xacro:property name="torpedo" value="${config['torpedoes']}"/>
     <joint name="${namespace}/torpedo_joint" type="fixed">
       <origin xyz="${torpedo['pose'][0]} ${torpedo['pose'][1]} ${torpedo['pose'][2]}"
@@ -92,12 +92,18 @@
         thrusters="${config['thrusters']}"
         index="0"/>
-  <xacro:poker_macro
-        namespace="${namespace}"
-        config="${config}"/>
-  <xacro:torpedo_macro
-        namespace="${namespace}"
-        config="${config}"/>
-  <xacro:dropper_macro
-        namespace="${namespace}"
-        config="${config}"/>
+  <xacro:if value="${'poker' in config}">
+    <xacro:poker_macro
+          namespace="${namespace}"
+          config="${config}"/>
+  </xacro:if>
+  <xacro:if value="${'torpedoes' in config}">
+    <xacro:torpedo_macro
+          namespace="${namespace}"
+          config="${config}"/>
+  </xacro:if>
+  <xacro:if value="${'droppers' in config}">
+    <xacro:dropper_macro
+          namespace="${namespace}"
+          config="${config}"/>
+  </xacro:if>
 </robot>

File: riptide_descriptions/urdf/robot_base.xacro (robot description, xacro)
@@ -3,5 +3,4 @@
 <robot xmlns:xacro="http://www.ros.org/wiki/xacro" >
   <xacro:include filename="$(find riptide_descriptions2)/urdf/snippets.xacro" />
-  <xacro:include filename="$(find riptide_descriptions2)/urdf/robot.gazebo.xacro" />
   <xacro:macro name="robot_base"
     params="namespace config inertial_reference_frame">

File: riptide_descriptions/urdf/robot_sensors.xacro (robot description, xacro)
@@ -4,6 +4,5 @@
   <xacro:property name="dvl" value="${config['dvl']}"/>
   <!-- DVL  -->
-  <!-- TODO: restore below if when xacro releases 1.14.4 -->
-  <!-- <xacro:if value="${'dvl' in config}"> -->
+  <xacro:if value="${'dvl' in config}">
     <xacro:property name="dvl" value="${config['dvl']}"/>
     <xacro:dvl_plugin_macro
@@ -14,8 +13,8 @@
               rpy="${dvl['pose'][3]} ${dvl['pose'][4]} ${dvl['pose'][5]}"/>
     </xacro:dvl_plugin_macro>
-  <!-- </xacro:if> -->
+  </xacro:if>
   <!-- Pressure  -->
   <!-- TODO: restore below if when xacro releases 1.14.4 -->
-  <!-- <xacro:if value="${'depth' in config}"> -->
+  <xacro:if value="${'depth' in config}">
     <xacro:property name="depth" value="${config['depth']}"/>
     <xacro:pressure_plugin_macro
@@ -26,34 +25,38 @@
               rpy="${depth['pose'][3]} ${depth['pose'][4]} ${depth['pose'][5]}"/>
     </xacro:pressure_plugin_macro>
-  <!-- </xacro:if> -->
-  <!-- port acoustic pod -->
-  <xacro:property name="acoustics_port" value="${config['acoustics']['port']}"/>
-  <xacro:acoustics_plugin_macro
+  </xacro:if>
+  <xacro:if value="${'acoustics' in config}">
+    <!-- port acoustic pod -->
+    <xacro:property name="acoustics_port" value="${config['acoustics']['port']}"/>
+    <xacro:acoustics_plugin_macro
+      namespace="${namespace}"
+      suffix="_port"
+      parent_link="${namespace}/origin">
+      <origin xyz="${acoustics_port['pose'][0]} ${acoustics_port['pose'][1]} ${acoustics_port['pose'][2]}"
+              rpy="${acoustics_port['pose'][3]} ${acoustics_port['pose'][4]} ${acoustics_port['pose'][5]}"/>
+    </xacro:acoustics_plugin_macro>
+    <!--starboard acoustic pod-->
+    <xacro:property name="acoustics_starboard" value="${config['acoustics']['starboard']}"/>
+    <xacro:acoustics_plugin_macro
     namespace="${namespace}"
-    suffix="_port"
+    suffix="_starboard"
     parent_link="${namespace}/origin">
-    <origin xyz="${acoustics_port['pose'][0]} ${acoustics_port['pose'][1]} ${acoustics_port['pose'][2]}"
-            rpy="${acoustics_port['pose'][3]} ${acoustics_port['pose'][4]} ${acoustics_port['pose'][5]}"/>
-  </xacro:acoustics_plugin_macro>
-  <!--starboard acoustic pod-->
-  <xacro:property name="acoustics_starboard" value="${config['acoustics']['starboard']}"/>
-  <xacro:acoustics_plugin_macro
-  namespace="${namespace}"
-  suffix="_starboard"
-  parent_link="${namespace}/origin">
-  <origin xyz="${acoustics_starboard['pose'][0]} ${acoustics_starboard['pose'][1]} ${acoustics_starboard['pose'][2]}"
-          rpy="${acoustics_starboard['pose'][3]} ${acoustics_starboard['pose'][4]} ${acoustics_starboard['pose'][5]}"/>
-  </xacro:acoustics_plugin_macro>
-  <xacro:property name="fog" value="${config['fog']}"/>
-  <xacro:fog_plugin_macro
-  namespace="${namespace}"
-  parent_link="${namespace}/origin">
-  <origin xyz="${fog['pose'][0]} ${fog['pose'][1]} ${fog['pose'][2]}"
-          rpy="${fog['pose'][3]} ${fog['pose'][4]} ${fog['pose'][5]}"/>
-  </xacro:fog_plugin_macro>
+    <origin xyz="${acoustics_starboard['pose'][0]} ${acoustics_starboard['pose'][1]} ${acoustics_starboard['pose'][2]}"
+            rpy="${acoustics_starboard['pose'][3]} ${acoustics_starboard['pose'][4]} ${acoustics_starboard['pose'][5]}"/>
+    </xacro:acoustics_plugin_macro>
+  </xacro:if>
+  <!-- Fiber Optic Gyro -->
+  <xacro:if value="${'fog' in config}">
+    <xacro:property name="fog" value="${config['fog']}"/>
+    <xacro:fog_plugin_macro
+    namespace="${namespace}"
+    parent_link="${namespace}/origin">
+    <origin xyz="${fog['pose'][0]} ${fog['pose'][1]} ${fog['pose'][2]}"
+            rpy="${fog['pose'][3]} ${fog['pose'][4]} ${fog['pose'][5]}"/>
+    </xacro:fog_plugin_macro>
+  </xacro:if>
   <!-- IMU  -->
   <!-- TODO: Get imu model from config -->
-  <!-- TODO: restore below if when xacro releases 1.14.4 -->
-  <!-- <xacro:if value="${'imu' in config}"> -->
+  <xacro:if value="${'imu' in config}">
     <xacro:property name="imu" value="${config['imu']}"/>
     <xacro:imu_plugin_macro
@@ -64,5 +67,5 @@
               rpy="${imu['pose'][3]} ${imu['pose'][4]} ${imu['pose'][5]}"/>
     </xacro:imu_plugin_macro>
-  <!-- </xacro:if> -->
+  </xacro:if>
   <!-- Pose sensor as ground truth for state estimation -->
   <xacro:default_pose_3d_macro

Commit message: added the tank hitch to talos

File: riptide_descriptions/urdf/robot_actuators.xacro (robot description, xacro)
@@ -30,18 +30,9 @@
     </xacro:if>
   </xacro:macro>
-  <xacro:macro name="poker_macro" params="namespace config">
-    <xacro:property name="poker" value="${config['poker']}"/>
-    <joint name="${namespace}/poker_joint" type="fixed">
-      <origin xyz="${poker['pose'][0]} ${poker['pose'][1]} ${poker['pose'][2]}"
-              rpy="${poker['pose'][3]} ${poker['pose'][4]} ${poker['pose'][5]}"/>
-      <parent link="${namespace}/origin"/>
-      <child link="${namespace}/poker_link"/>
-    </joint>
-    <link name="${namespace}/poker_link">
-      <xacro:dummy_inertia />
-      <xacro:no_collision />
-    </link>
+  <xacro:macro name="origin_from_pose_macro" params="pose">
+    <origin xyz="${pose[0]} ${pose[1]} ${pose[2]}"
+            rpy="${pose[3]} ${pose[4]} ${pose[5]}" />
   </xacro:macro>
-  <xacro:macro name="launcher_macro" params="namespace name parent *origin">
+  <xacro:macro name="generic_link_macro_with_origin" params="namespace name parent *origin">
     <link name="${namespace}/${name}_link">
       <xacro:dummy_inertia/>
@@ -49,42 +40,25 @@
     </link>
     <joint name="${namespace}/${name}_joint" type="fixed">
-      <xacro:insert_block name="origin"/>
+      <xacro:insert_block name="origin" />
       <parent link="${parent}"/>
       <child link="${namespace}/${name}_link"/>
     </joint>
   </xacro:macro>
+  <xacro:macro name="generic_link_macro" params="namespace name parent pose">
+    <xacro:generic_link_macro_with_origin namespace="${namespace}" name="${name}" parent="${parent}">
+      <xacro:origin_from_pose_macro pose="${pose}" />
+    </xacro:generic_link_macro_with_origin>
+  </xacro:macro>
   <xacro:macro name="torpedo_macro" params="namespace config">
     <xacro:property name="torpedo" value="${config['torpedoes']}"/>
-    <joint name="${namespace}/torpedo_joint" type="fixed">
-      <origin xyz="${torpedo['pose'][0]} ${torpedo['pose'][1]} ${torpedo['pose'][2]}"
-              rpy="${torpedo['pose'][3]} ${torpedo['pose'][4]} ${torpedo['pose'][5]}" />
-      <parent link="${namespace}/origin"/>
-      <child link="${namespace}/torpedo_link"/>
-    </joint>
-    <link name="${namespace}/torpedo_link">
-      <xacro:dummy_inertia />
-      <xacro:no_collision />
-    </link>
-    <xacro:launcher_macro namespace="${namespace}" name="torpedo_0" parent="${namespace}/torpedo_link">
+    <xacro:generic_link_macro namespace="${namespace}" name="torpedo" parent="${namespace}/origin" pose="${torpedo['pose']}" />
+    <xacro:generic_link_macro_with_origin namespace="${namespace}" name="torpedo_0" parent="${namespace}/torpedo_link">
       <origin xyz="0 ${-torpedo['baseline'] / 2} 0"
               rpy="0 0 0"/>
-    </xacro:launcher_macro>
-    <xacro:launcher_macro namespace="${namespace}" name="torpedo_1" parent="${namespace}/torpedo_link">
+    </xacro:generic_link_macro_with_origin>
+    <xacro:generic_link_macro_with_origin namespace="${namespace}" name="torpedo_1" parent="${namespace}/torpedo_link">
       <origin xyz="0 ${torpedo['baseline'] / 2} 0"
               rpy="0 0 0"/>
-    </xacro:launcher_macro>
-  </xacro:macro>
-  <xacro:macro name="dropper_macro" params="namespace config">
-    <xacro:property name="dropper" value="${config['droppers']}"/>
-    <joint name="${namespace}/dropper_joint" type="fixed">
-      <origin xyz="${dropper['pose'][0]} ${dropper['pose'][1]} ${dropper['pose'][2]}"
-              rpy="${dropper['pose'][3]} ${dropper['pose'][4]} ${dropper['pose'][5]}" />
-      <parent link="${namespace}/origin"/>
-      <child link="${namespace}/droppers_link"/>
-    </joint>
-    <link name="${namespace}/droppers_link">
-      <xacro:dummy_inertia />
-      <xacro:no_collision />
-    </link>
+    </xacro:generic_link_macro_with_origin>
   </xacro:macro>
   <xacro:thrusters_macro
@@ -93,7 +67,9 @@
         index="0"/>
   <xacro:if value="${'poker' in config}">
-    <xacro:poker_macro
+    <xacro:generic_link_macro
           namespace="${namespace}"
-          config="${config}"/>
+          name="poker"
+          parent="${namespace}/origin"
+          pose="${config['poker']['pose']}" />
   </xacro:if>
   <xacro:if value="${'torpedoes' in config}">
@@ -103,7 +79,16 @@
   </xacro:if>
   <xacro:if value="${'droppers' in config}">
-    <xacro:dropper_macro
+    <xacro:generic_link_macro
           namespace="${namespace}"
-          config="${config}"/>
+          name="droppers"
+          parent="${namespace}/origin"
+          pose="${config['droppers']['pose']}" />
+  </xacro:if>
+  <xacro:if value="${'hitch' in config}">
+    <xacro:generic_link_macro
+          namespace="${namespace}"
+          name="hitch"
+          parent="${namespace}/origin"
+          pose="${config['hitch']['pose']}" />
   </xacro:if>
 </robot>
